File: ESP32ControlStand/ButtonLEDPanel.sch (KiCad schematic (older format))
At the start: 24 parts, among them P201 CONN_5, SW201 SW_PUSH_SMALL, SW202 SW_PUSH_SMALL, SW203 SW_PUSH_SMALL, SW204 SW_PUSH_SMALL, SW205 SW_PUSH_SMALL, SW206 SW_PUSH_SMALL, SW207 SW_PUSH_SMALL, SW208 SW_PUSH_SMALL, T201 Buttons, T202 LEDS, U201 MCP23017, U202 TBD62083A

Commit message: Continue FreeCAD work
Parts:
- C201: symbol C -> C-RESCUE-ESP32ControlStand
- D201, D202, D203, D204, D205, D206, D207, D208: symbol LED -> LED-RESCUE-ESP32ControlStand
- R201: symbol R -> R-RESCUE-ESP32ControlStand
- U201: symbol MCP23017 -> MCP23017-RESCUE-ESP32ControlStand
Connections:
- net +3.3V: now also R201.1
- net at U201.18 (Reset): now also R201.2
Changed lines of the file:
@@
 EESchema Schematic File Version 2
+LIBS:ESP32ControlStand-rescue
 LIBS:power
 LIBS:device
@@
 LIBS:memory
 LIBS:xilinx
-LIBS:special
 LIBS:microcontrollers
 LIBS:dsp
@@
 LIBS:adafruit_powerboost_500
 LIBS:ESP32ControlStand-cache
-EELAYER 27 0
+EELAYER 25 0
 EELAYER END
 $Descr A4 11693 8268
@@
 $EndDescr
 $Comp
-L MCP23017 U201
+L MCP23017-RESCUE-ESP32ControlStand U201
 U 1 1 5D93EF0F
 P 4100 2400
@@
 	5950 3400 5950 3650
 $Comp
-L GND #PWR024
+L GND-RESCUE-ESP32ControlStand #PWR024
 U 1 1 5D93F4A1
 P 5950 3650
@@
 Connection ~ 5950 3500
 $Comp
-L LED D201
+L LED-RESCUE-ESP32ControlStand D201
 U 1 1 5D93F5DD
 P 10150 1050
@@
 $EndComp
 $Comp
-L LED D202
+L LED-RESCUE-ESP32ControlStand D202
 U 1 1 5D93F5EC
 P 10150 1450
@@
 $EndComp
 $Comp
-L LED D203
+L LED-RESCUE-ESP32ControlStand D203
 U 1 1 5D93F5FB
 P 10150 1850
@@
 $EndComp
 $Comp
-L LED D204
+L LED-RESCUE-ESP32ControlStand D204
 U 1 1 5D93F60A
 P 10150 2250
@@
 $EndComp
 $Comp
-L LED D205
+L LED-RESCUE-ESP32ControlStand D205
 U 1 1 5D93F619
 P 10150 2600
@@
 $EndComp
 $Comp
-L LED D206
+L LED-RESCUE-ESP32ControlStand D206
 U 1 1 5D93F628
 P 10150 3000
@@
 $EndComp
 $Comp
-L LED D207
+L LED-RESCUE-ESP32ControlStand D207
 U 1 1 5D93F637
 P 10150 3400
@@
 $EndComp
 $Comp
-L LED D208
+L LED-RESCUE-ESP32ControlStand D208
 U 1 1 5D93F646
 P 10150 3800
@@
 $EndComp
 $Comp
-L GND #PWR026
+L GND-RESCUE-ESP32ControlStand #PWR026
 U 1 1 5D93F67D
 P 8000 4200
@@
 Connection ~ 10350 1050
 $Comp
-L GND #PWR028
+L GND-RESCUE-ESP32ControlStand #PWR028
 U 1 1 5D94002B
 P 4000 3850
@@
 	4000 3650 4000 3850
 $Comp
-L +3.3V #PWR029
+L +3.3V-RESCUE-ESP32ControlStand #PWR029
 U 1 1 5D94010D
 P 4100 1000
@@
 Connection ~ 3400 1950
 $Comp
-L GND #PWR030
+L GND-RESCUE-ESP32ControlStand #PWR030
 U 1 1 5D94025D
 P 3400 2200
@@
 Connection ~ 3400 2050
 $Comp
-L R R201
+L R-RESCUE-ESP32ControlStand R201
 U 1 1 5D940347
 P 3050 2850
@@
 $EndComp
 $Comp
-L +3.3V #PWR031
+L +3.3V-RESCUE-ESP32ControlStand #PWR031
 U 1 1 5D94035B
 P 2600 2850
@@
 $EndComp
 $Comp
-L +3.3V #PWR033
+L +3.3V-RESCUE-ESP32ControlStand #PWR033
 U 1 1 5D94046A
 P 2750 1550
@@
 $EndComp
 $Comp
-L GND #PWR034
+L GND-RESCUE-ESP32ControlStand #PWR034
 U 1 1 5D94049C
 P 2800 1700
@@
 NoConn ~ 3400 2650
 $Comp
-L C C201
+L C-RESCUE-ESP32ControlStand C201
 U 1 1 5D95DF47
 P 2750 2350
