File: ESP32ControlStand/CAN_Transceiver.sch (KiCad schematic (older format))
At the start: 14 parts, among them J401 RJ45, J402 RJ45, T401 + 15 in -, T402 + 15 out -, U401 TCAN332DR, U402 SN65HVD233-HT

Commit message: Continue FreeCAD work
Parts:
- C401, C403: symbol C -> C-RESCUE-ESP32ControlStand
- C402: symbol CP1 -> CP1-RESCUE-ESP32ControlStand
- R401, R402: symbol R -> R-RESCUE-ESP32ControlStand
Changed lines of the file:
@@
 EESchema Schematic File Version 2
+LIBS:ESP32ControlStand-rescue
 LIBS:power
 LIBS:device
@@
 LIBS:memory
 LIBS:xilinx
-LIBS:special
 LIBS:microcontrollers
 LIBS:dsp
@@
 LIBS:adafruit_powerboost_500
 LIBS:ESP32ControlStand-cache
-EELAYER 27 0
+EELAYER 25 0
 EELAYER END
 $Descr A4 11693 8268
@@
 $EndComp
 $Comp
-L +3.3V #PWR046
+L +3.3V-RESCUE-ESP32ControlStand #PWR046
 U 1 1 5D94A57B
 P 4100 2900
@@
 $EndComp
 $Comp
-L +3.3V #PWR047
+L +3.3V-RESCUE-ESP32ControlStand #PWR047
 U 1 1 5D94A57C
 P 4100 4050
@@
 $EndComp
 $Comp
-L GND #PWR048
+L GND-RESCUE-ESP32ControlStand #PWR048
 U 1 1 5D94A57D
 P 4100 3800
@@
 $EndComp
 $Comp
-L GND #PWR049
+L GND-RESCUE-ESP32ControlStand #PWR049
 U 1 1 5D94A57E
 P 4100 4950
@@
 Connection ~ 3750 4400
 $Comp
-L C C401
+L C-RESCUE-ESP32ControlStand C401
 U 1 1 5D94A57F
 P 4650 3800
@@
 $EndComp
 $Comp
-L CP1 C402
+L CP1-RESCUE-ESP32ControlStand C402
 U 1 1 5D94A580
 P 5000 3800
@@
 CANL
 $Comp
-L R R401
+L R-RESCUE-ESP32ControlStand R401
 U 1 1 5D94A581
 P 5850 3650
@@
 $EndComp
 $Comp
-L R R402
+L R-RESCUE-ESP32ControlStand R402
 U 1 1 5D94A582
 P 6550 3650
@@
 	6700 4150 6600 4150
 $Comp
-L C C403
+L C-RESCUE-ESP32ControlStand C403
 U 1 1 5D94A584
 P 6200 4750
@@
 $EndComp
 $Comp
-L GND #PWR050
+L GND-RESCUE-ESP32ControlStand #PWR050
 U 1 1 5D94A585
 P 6200 5100
@@
 	7450 3000 7450 5050
 $Comp
-L GND #PWR051
+L GND-RESCUE-ESP32ControlStand #PWR051
 U 1 1 5D94A58A
 P 6750 2650
