File: ESP32ControlStand/PowerSupply.sch (KiCad schematic (older format))
At the start: 5 parts, among them U501 LM2574N-5.0

Commit message: Continue FreeCAD work
Parts:
- C501, C502: symbol CP1 -> CP1-RESCUE-ESP32ControlStand
Changed lines of the file:
@@
 EESchema Schematic File Version 2
+LIBS:ESP32ControlStand-rescue
 LIBS:power
 LIBS:device
@@
 LIBS:memory
 LIBS:xilinx
-LIBS:special
 LIBS:microcontrollers
 LIBS:dsp
@@
 LIBS:adafruit_powerboost_500
 LIBS:ESP32ControlStand-cache
-EELAYER 27 0
+EELAYER 25 0
 EELAYER END
 $Descr A4 11693 8268
@@
 $EndComp
 $Comp
-L CP1 C502
+L CP1-RESCUE-ESP32ControlStand C502
 U 1 1 5D94AA5A
 P 5950 2900
@@
 $EndComp
 $Comp
-L CP1 C501
+L CP1-RESCUE-ESP32ControlStand C501
 U 1 1 5D94AA5B
 P 3700 2800
@@
 Connection ~ 4850 3300
 $Comp
-L GND #PWR053
+L GND-RESCUE-ESP32ControlStand #PWR053
 U 1 1 5D94AA5E
 P 4850 3400
