File: ESP32-D0WD-V3-ControlStand/ButtonLedPanel2.sch (KiCad schematic (older format))
At the start: 25 parts, among them P9 CONN_5, SW15 SW_PUSH_SMALL, SW16 SW_PUSH_SMALL, SW17 SW_PUSH_SMALL, SW18 SW_PUSH_SMALL, SW19 SW_PUSH_SMALL, SW20 SW_PUSH_SMALL, SW21 SW_PUSH_SMALL, SW22 SW_PUSH_SMALL, T3 Buttons, T4 LEDS, U3 MCP23017, U4 TBD62083A

Commit message: Working on the PCB Layout.
Parts:
- added MK13, MK14, MK15, MK16: Mounting_Hole, Mounting_Holes:MountingHole_2.5mm, symbol Mounting_Hole
- U4: footprint ~ -> Housings_SOIC:SOIC-18W_7.5x11.6mm_Pitch1.27mm
Changed lines of the file:
@@
 LIBS:mcp73871
 LIBS:lm2574n-5
+LIBS:mechanical
+LIBS:graphic_symbols
 LIBS:ESP32-D0WD-V3-ControlStand-cache
 EELAYER 25 0
@@
 F 0 "U4" H 8100 1300 60  0000 C CNN
 F 1 "TBD62083A" H 8250 1550 60  0000 C CNN
-F 2 "~" H 8000 1450 60  0000 C CNN
+F 2 "Housings_SOIC:SOIC-18W_7.5x11.6mm_Pitch1.27mm" H 8000 1450 60  0001 C CNN
 F 3 "~" H 8000 1450 60  0000 C CNN
 	2    8000 1450
@@
 F 0 "U4" H 8100 1700 60  0000 C CNN
 F 1 "TBD62083A" H 8250 1950 60  0000 C CNN
-F 2 "~" H 8000 1850 60  0000 C CNN
+F 2 "Housings_SOIC:SOIC-18W_7.5x11.6mm_Pitch1.27mm" H 8000 1850 60  0001 C CNN
 F 3 "~" H 8000 1850 60  0000 C CNN
 	3    8000 1850
@@
 F 0 "U4" H 8100 2100 60  0000 C CNN
 F 1 "TBD62083A" H 8250 2350 60  0000 C CNN
-F 2 "~" H 8000 2250 60  0000 C CNN
+F 2 "Housings_SOIC:SOIC-18W_7.5x11.6mm_Pitch1.27mm" H 8000 2250 60  0001 C CNN
 F 3 "~" H 8000 2250 60  0000 C CNN
 	4    8000 2250
@@
 F 0 "U4" H 8100 2450 60  0000 C CNN
 F 1 "TBD62083A" H 8250 2700 60  0000 C CNN
-F 2 "~" H 8000 2600 60  0000 C CNN
+F 2 "Housings_SOIC:SOIC-18W_7.5x11.6mm_Pitch1.27mm" H 8000 2600 60  0001 C CNN
 F 3 "~" H 8000 2600 60  0000 C CNN
 	5    8000 2600
@@
 F 0 "U4" H 8100 2850 60  0000 C CNN
 F 1 "TBD62083A" H 8250 3100 60  0000 C CNN
-F 2 "~" H 8000 3000 60  0000 C CNN
+F 2 "Housings_SOIC:SOIC-18W_7.5x11.6mm_Pitch1.27mm" H 8000 3000 60  0001 C CNN
 F 3 "~" H 8000 3000 60  0000 C CNN
 	6    8000 3000
@@
 F 0 "U4" H 8100 3250 60  0000 C CNN
 F 1 "TBD62083A" H 8250 3500 60  0000 C CNN
-F 2 "~" H 8000 3400 60  0000 C CNN
+F 2 "Housings_SOIC:SOIC-18W_7.5x11.6mm_Pitch1.27mm" H 8000 3400 60  0001 C CNN
 F 3 "~" H 8000 3400 60  0000 C CNN
 	7    8000 3400
@@
 F 0 "U4" H 8100 3650 60  0000 C CNN
 F 1 "TBD62083A" H 8250 3900 60  0000 C CNN
-F 2 "~" H 8000 3800 60  0000 C CNN
+F 2 "Housings_SOIC:SOIC-18W_7.5x11.6mm_Pitch1.27mm" H 8000 3800 60  0001 C CNN
 F 3 "~" H 8000 3800 60  0000 C CNN
 	8    8000 3800
@@
 	5950 3400 5950 3650
 $Comp
-L GND-RESCUE-ESP32ControlStand #PWR36
+L GND-RESCUE-ESP32ControlStand #PWR029
 U 1 1 62DF18E6
 P 5950 3650
-F 0 "#PWR36" H 5950 3650 30  0001 C CNN
+F 0 "#PWR029" H 5950 3650 30  0001 C CNN
 F 1 "GND" H 5950 3580 30  0001 C CNN
 F 2 "" H 5950 3650 60  0000 C CNN
@@
 $EndComp
 $Comp
-L +BATT #PWR37
+L +BATT #PWR030
 U 1 1 62DF18F0
 P 8000 750
-F 0 "#PWR37" H 8000 700 20  0001 C CNN
+F 0 "#PWR030" H 8000 700 20  0001 C CNN
 F 1 "+BATT" H 8000 850 30  0000 C CNN
 F 2 "" H 8000 750 60  0000 C CNN
@@
 $EndComp
 $Comp
-L GND-RESCUE-ESP32ControlStand #PWR38
+L GND-RESCUE-ESP32ControlStand #PWR031
 U 1 1 62DF18F1
 P 8000 4200
-F 0 "#PWR38" H 8000 4200 30  0001 C CNN
+F 0 "#PWR031" H 8000 4200 30  0001 C CNN
 F 1 "GND" H 8000 4130 30  0001 C CNN
 F 2 "" H 8000 4200 60  0000 C CNN
@@
 $EndComp
 $Comp
-L +BATT #PWR39
+L +BATT #PWR032
 U 1 1 62DF18F2
 P 10500 650
-F 0 "#PWR39" H 10500 600 20  0001 C CNN
+F 0 "#PWR032" H 10500 600 20  0001 C CNN
 F 1 "+BATT" H 10500 750 30  0000 C CNN
 F 2 "" H 10500 650 60  0000 C CNN
@@
 Connection ~ 10350 1050
 $Comp
-L GND-RESCUE-ESP32ControlStand #PWR34
+L GND-RESCUE-ESP32ControlStand #PWR033
 U 1 1 62DF18F3
 P 4000 3850
-F 0 "#PWR34" H 4000 3850 30  0001 C CNN
+F 0 "#PWR033" H 4000 3850 30  0001 C CNN
 F 1 "GND" H 4000 3780 30  0001 C CNN
 F 2 "" H 4000 3850 60  0000 C CNN
@@
 	4000 3650 4000 3850
 $Comp
-L +3.3V-RESCUE-ESP32ControlStand #PWR35
+L +3.3V-RESCUE-ESP32ControlStand #PWR034
 U 1 1 62DF18F4
 P 4100 1000
-F 0 "#PWR35" H 4100 960 30  0001 C CNN
+F 0 "#PWR034" H 4100 960 30  0001 C CNN
 F 1 "+3.3V" H 4100 1110 30  0000 C CNN
 F 2 "" H 4100 1000 60  0000 C CNN
@@
 	4100 1000 4100 1200
 $Comp
-L GND-RESCUE-ESP32ControlStand #PWR33
+L GND-RESCUE-ESP32ControlStand #PWR035
 U 1 1 62DF18F5
 P 3250 1850
-F 0 "#PWR33" H 3250 1850 30  0001 C CNN
+F 0 "#PWR035" H 3250 1850 30  0001 C CNN
 F 1 "GND" H 3250 1780 30  0001 C CNN
 F 2 "" H 3250 1850 60  0000 C CNN
@@
 $EndComp
 $Comp
-L +3.3V-RESCUE-ESP32ControlStand #PWR29
+L +3.3V-RESCUE-ESP32ControlStand #PWR036
 U 1 1 62DF18F7
 P 2600 2850
-F 0 "#PWR29" H 2600 2810 30  0001 C CNN
+F 0 "#PWR036" H 2600 2810 30  0001 C CNN
 F 1 "+3.3V" H 2600 2960 30  0000 C CNN
 F 2 "" H 2600 2850 60  0000 C CNN
@@
 $EndComp
 $Comp
-L +BATT #PWR30
+L +BATT #PWR037
 U 1 1 62DF18F9
 P 2750 1400
-F 0 "#PWR30" H 2750 1350 20  0001 C CNN
+F 0 "#PWR037" H 2750 1350 20  0001 C CNN
 F 1 "+BATT" H 2750 1500 30  0000 C CNN
 F 2 "" H 2750 1400 60  0000 C CNN
@@
 $EndComp
 $Comp
-L +3.3V-RESCUE-ESP32ControlStand #PWR31
+L +3.3V-RESCUE-ESP32ControlStand #PWR038
 U 1 1 62DF18FA
 P 2750 1550
-F 0 "#PWR31" H 2750 1510 30  0001 C CNN
+F 0 "#PWR038" H 2750 1510 30  0001 C CNN
 F 1 "+3.3V" H 2750 1660 30  0000 C CNN
 F 2 "" H 2750 1550 60  0000 C CNN
@@
 $EndComp
 $Comp
-L GND-RESCUE-ESP32ControlStand #PWR32
+L GND-RESCUE-ESP32ControlStand #PWR039
 U 1 1 62DF18FB
 P 2800 1700
-F 0 "#PWR32" H 2800 1700 30  0001 C CNN
+F 0 "#PWR039" H 2800 1700 30  0001 C CNN
 F 1 "GND" H 2800 1630 30  0001 C CNN
 F 2 "" H 2800 1700 60  0000 C CNN
@@
 F 0 "R8" V 3130 2050 40  0000 C CNN
 F 1 "10K" V 3057 2051 40  0000 C CNN
-F 2 "Resistors_SMD:R_0402" V 2980 2050 30  0000 C CNN
+F 2 "Resistors_SMD:R_0402" V 2980 2050 30  0001 C CNN
 F 3 "~" H 3050 2050 30  0000 C CNN
 F 4 "603-RC0402JR-0710KL" V 3050 2050 60  0001 C CNN "Mouser Part Number"
@@
 	3350 2250 3350 1850
 Connection ~ 3350 1850
+$Comp
+L Mounting_Hole MK15
+U 1 1 62E6E676
+P 6850 3350
+F 0 "MK15" H 6850 3550 50  0000 C CNN
+F 1 "Mounting_Hole" H 6850 3475 50  0000 C CNN
+F 2 "Mounting_Holes:MountingHole_2.5mm" H 6850 3350 50  0001 C CNN
+F 3 "" H 6850 3350 50  0001 C CNN
+	1    6850 3350
+	1    0    0    -1
+$EndComp
+$Comp
+L Mounting_Hole MK16
+U 1 1 62E6E6F9
+P 6950 3650
+F 0 "MK16" H 6950 3850 50  0000 C CNN
+F 1 "Mounting_Hole" H 6950 3775 50  0000 C CNN
+F 2 "Mounting_Holes:MountingHole_2.5mm" H 6950 3650 50  0001 C CNN
+F 3 "" H 6950 3650 50  0001 C CNN
+	1    6950 3650
+	1    0    0    -1
+$EndComp
+$Comp
+L Mounting_Hole MK14
+U 1 1 62E6E752
+P 6750 3850
+F 0 "MK14" H 6750 4050 50  0000 C CNN
+F 1 "Mounting_Hole" H 6750 3975 50  0000 C CNN
+F 2 "Mounting_Holes:MountingHole_2.5mm" H 6750 3850 50  0001 C CNN
+F 3 "" H 6750 3850 50  0001 C CNN
+	1    6750 3850
+	1    0    0    -1
+$EndComp
+$Comp
+L Mounting_Hole MK13
+U 1 1 62E6E7B1
+P 6450 4000
+F 0 "MK13" H 6450 4200 50  0000 C CNN
+F 1 "Mounting_Hole" H 6450 4125 50  0000 C CNN
+F 2 "Mounting_Holes:MountingHole_2.5mm" H 6450 4000 50  0001 C CNN
+F 3 "" H 6450 4000 50  0001 C CNN
+	1    6450 4000
+	1    0    0    -1
+$EndComp
 $EndSCHEMATC

Commit message: Completed V0.0 PCB.
Connections:
- net +3.3V renamed +3V3
Changed lines of the file:
@@
 	5950 3400 5950 3650
 $Comp
-L GND-RESCUE-ESP32ControlStand #PWR029
+L GND #PWR031
 U 1 1 62DF18E6
 P 5950 3650
-F 0 "#PWR029" H 5950 3650 30  0001 C CNN
+F 0 "#PWR031" H 5950 3650 30  0001 C CNN
 F 1 "GND" H 5950 3580 30  0001 C CNN
 F 2 "" H 5950 3650 60  0000 C CNN
@@
 $EndComp
 $Comp
-L +BATT #PWR030
+L +BATT #PWR032
 U 1 1 62DF18F0
 P 8000 750
-F 0 "#PWR030" H 8000 700 20  0001 C CNN
+F 0 "#PWR032" H 8000 700 20  0001 C CNN
 F 1 "+BATT" H 8000 850 30  0000 C CNN
 F 2 "" H 8000 750 60  0000 C CNN
@@
 $EndComp
 $Comp
-L GND-RESCUE-ESP32ControlStand #PWR031
+L GND #PWR033
 U 1 1 62DF18F1
 P 8000 4200
-F 0 "#PWR031" H 8000 4200 30  0001 C CNN
+F 0 "#PWR033" H 8000 4200 30  0001 C CNN
 F 1 "GND" H 8000 4130 30  0001 C CNN
 F 2 "" H 8000 4200 60  0000 C CNN
@@
 $EndComp
 $Comp
-L +BATT #PWR032
+L +BATT #PWR034
 U 1 1 62DF18F2
 P 10500 650
-F 0 "#PWR032" H 10500 600 20  0001 C CNN
+F 0 "#PWR034" H 10500 600 20  0001 C CNN
 F 1 "+BATT" H 10500 750 30  0000 C CNN
 F 2 "" H 10500 650 60  0000 C CNN
@@
 Connection ~ 10350 1050
 $Comp
-L GND-RESCUE-ESP32ControlStand #PWR033
+L GND #PWR035
 U 1 1 62DF18F3
 P 4000 3850
-F 0 "#PWR033" H 4000 3850 30  0001 C CNN
+F 0 "#PWR035" H 4000 3850 30  0001 C CNN
 F 1 "GND" H 4000 3780 30  0001 C CNN
 F 2 "" H 4000 3850 60  0000 C CNN
@@
 	4000 3650 4000 3850
 $Comp
-L +3.3V-RESCUE-ESP32ControlStand #PWR034
+L +3.3V #PWR036
 U 1 1 62DF18F4
 P 4100 1000
-F 0 "#PWR034" H 4100 960 30  0001 C CNN
+F 0 "#PWR036" H 4100 960 30  0001 C CNN
 F 1 "+3.3V" H 4100 1110 30  0000 C CNN
 F 2 "" H 4100 1000 60  0000 C CNN
@@
 	4100 1000 4100 1200
 $Comp
-L GND-RESCUE-ESP32ControlStand #PWR035
+L GND #PWR037
 U 1 1 62DF18F5
 P 3250 1850
-F 0 "#PWR035" H 3250 1850 30  0001 C CNN
+F 0 "#PWR037" H 3250 1850 30  0001 C CNN
 F 1 "GND" H 3250 1780 30  0001 C CNN
 F 2 "" H 3250 1850 60  0000 C CNN
@@
 F 0 "R9" V 3130 2850 40  0000 C CNN
 F 1 "10K" V 3057 2851 40  0000 C CNN
-F 2 "Resistors_SMD:R_0402" V 2980 2850 30  0000 C CNN
+F 2 "Resistors_SMD:R_0402" V 2980 2850 30  0001 C CNN
 F 3 "~" H 3050 2850 30  0000 C CNN
 F 4 "603-RC0402JR-0710KL" V 3050 2850 60  0001 C CNN "Mouser Part Number"
@@
 $EndComp
 $Comp
-L +3.3V-RESCUE-ESP32ControlStand #PWR036
+L +3.3V #PWR038
 U 1 1 62DF18F7
 P 2600 2850
-F 0 "#PWR036" H 2600 2810 30  0001 C CNN
+F 0 "#PWR038" H 2600 2810 30  0001 C CNN
 F 1 "+3.3V" H 2600 2960 30  0000 C CNN
 F 2 "" H 2600 2850 60  0000 C CNN
@@
 $EndComp
 $Comp
-L +BATT #PWR037
+L +BATT #PWR039
 U 1 1 62DF18F9
 P 2750 1400
-F 0 "#PWR037" H 2750 1350 20  0001 C CNN
+F 0 "#PWR039" H 2750 1350 20  0001 C CNN
 F 1 "+BATT" H 2750 1500 30  0000 C CNN
 F 2 "" H 2750 1400 60  0000 C CNN
@@
 $EndComp
 $Comp
-L +3.3V-RESCUE-ESP32ControlStand #PWR038
+L +3.3V #PWR040
 U 1 1 62DF18FA
 P 2750 1550
-F 0 "#PWR038" H 2750 1510 30  0001 C CNN
+F 0 "#PWR040" H 2750 1510 30  0001 C CNN
 F 1 "+3.3V" H 2750 1660 30  0000 C CNN
 F 2 "" H 2750 1550 60  0000 C CNN
@@
 $EndComp
 $Comp
-L GND-RESCUE-ESP32ControlStand #PWR039
+L GND #PWR041
 U 1 1 62DF18FB
 P 2800 1700
-F 0 "#PWR039" H 2800 1700 30  0001 C CNN
+F 0 "#PWR041" H 2800 1700 30  0001 C CNN
 F 1 "GND" H 2800 1630 30  0001 C CNN
 F 2 "" H 2800 1700 60  0000 C CNN
