File: ESP32-D0WD-V3-ControlStand/ESP32-D0WD-V3-ControlStand.kicad_pcb (KiCad board)
At the start: 2 copper layers, 0 parts

Commit message: Transfer edge cuts.
Other:
- board outline added: 184.1 x 144.1 mm
Changed lines of the file:
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@@
     (links 0)
     (no_connects 0)
-    (area 0 0 0 0)
+    (area 30.430078 17.34908 214.679955 161.593984)
     (thickness 1.6)
-    (drawings 0)
+    (drawings 91)
     (tracks 0)
     (zones 0)
@@
     (uvia_drill 0.1)
   )
+  (gr_line (start 71.120051 29.464073) (end 57.785061 29.464073) (layer Edge.Cuts) (width 0.1))
+  (gr_line (start 83.185043 161.543983) (end 83.185043 148.843991) (layer Edge.Cuts) (width 0.1))
+  (gr_line (start 147.954999 17.399081) (end 214.629954 17.399081) (layer Edge.Cuts) (width 0.1))
+  (gr_line (start 80.645045 109.474018) (end 80.645045 96.774027) (layer Edge.Cuts) (width 0.1))
+  (gr_line (start 143.510002 122.809009) (end 146.05 122.809009) (layer Edge.Cuts) (width 0.1))
+  (gr_line (start 146.05 135.509) (end 147.32 135.509) (layer Edge.Cuts) (width 0.1))
+  (gr_line (start 45.720069 148.843991) (end 45.720069 150.113991) (layer Edge.Cuts) (width 0.1))
+  (gr_line (start 66.040055 118.999012) (end 63.500057 118.999012) (layer Edge.Cuts) (width 0.1))
+  (gr_line (start 214.629954 96.774027) (end 214.629954 161.543983) (layer Edge.Cuts) (width 0.1))
+  (gr_line (start 83.185043 161.543983) (end 143.510002 161.543983) (layer Edge.Cuts) (width 0.1))
+  (gr_line (start 106.680027 96.774027) (end 116.205021 96.774027) (layer Edge.Cuts) (width 0.1))
+  (gr_line (start 71.120051 86.614034) (end 30.480079 86.614034) (layer Edge.Cuts) (width 0.1))
+  (gr_line (start 63.500057 96.774027) (end 63.500057 91.059031) (layer Edge.Cuts) (width 0.1))
+  (gr_line (start 71.120051 37.084067) (end 71.120051 29.464073) (layer Edge.Cuts) (width 0.1))
+  (gr_line (start 147.32 67.564047) (end 141.622783 67.564047) (layer Edge.Cuts) (width 0.1))
+  (gr_line (start 143.510002 161.543983) (end 143.510002 148.843991) (layer Edge.Cuts) (width 0.1))
+  (gr_line (start 74.295049 91.059031) (end 74.295049 67.564047) (layer Edge.Cuts) (width 0.1))
+  (gr_line (start 45.720069 118.999012) (end 31.750078 118.999012) (layer Edge.Cuts) (width 0.1))
+  (gr_line (start 64.770056 44.704062) (end 64.770056 61.214051) (layer Edge.Cuts) (width 0.1))
+  (gr_line (start 66.040055 109.474018) (end 63.500057 109.474018) (layer Edge.Cuts) (width 0.1))
+  (gr_line (start 214.629954 17.399081) (end 214.629954 91.059031) (layer Edge.Cuts) (width 0.1))
+  (gr_line (start 143.510002 109.474018) (end 143.510002 96.774027) (layer Edge.Cuts) (width 0.1))
+  (gr_line (start 74.295049 17.399081) (end 74.295049 39.624066) (layer Edge.Cuts) (width 0.1))
+  (gr_line (start 116.205021 92.964029) (end 116.205021 91.059031) (layer Edge.Cuts) (width 0.1))
+  (gr_line (start 147.32 91.059031) (end 147.32 67.564047) (layer Edge.Cuts) (width 0.1))
+  (gr_line (start 141.605004 17.399081) (end 141.605004 39.624066) (layer Edge.Cuts) (width 0.1))
+  (gr_line (start 31.750078 118.999012) (end 31.750078 91.059031) (layer Edge.Cuts) (width 0.1))
+  (gr_line (start 106.680027 96.774027) (end 93.980036 96.774027) (layer Edge.Cuts) (width 0.1))
+  (gr_line (start 80.645045 161.543983) (end 66.040055 161.543983) (layer Edge.Cuts) (width 0.1))
+  (gr_line (start 71.120051 39.624066) (end 71.120051 37.084067) (layer Edge.Cuts) (width 0.1))
+  (gr_line (start 63.500057 161.543983) (end 63.500057 148.843991) (layer Edge.Cuts) (width 0.1))
+  (gr_line (start 45.720069 133.604002) (end 45.720069 148.843991) (layer Edge.Cuts) (width 0.1))
+  (gr_line (start 45.720069 118.999012) (end 62.865057 118.999012) (layer Edge.Cuts) (width 0.1))
+  (gr_line (start 147.32 17.399081) (end 147.954999 17.399081) (layer Edge.Cuts) (width 0.1))
+  (gr_line (start 116.205021 91.059031) (end 74.295049 91.059031) (layer Edge.Cuts) (width 0.1))
+  (gr_line (start 128.905012 96.774027) (end 128.905012 92.964029) (layer Edge.Cuts) (width 0.1))
+  (gr_line (start 176.52998 96.774027) (end 176.52998 92.964029) (layer Edge.Cuts) (width 0.1))
+  (gr_line (start 80.645045 148.843991) (end 80.645045 161.543983) (layer Edge.Cuts) (width 0.1))
+  (gr_line (start 189.229971 91.059031) (end 214.629954 91.059031) (layer Edge.Cuts) (width 0.1))
+  (gr_line (start 71.120051 86.614034) (end 71.120051 67.564047) (layer Edge.Cuts) (width 0.1))
+  (gr_line (start 45.720069 132.969002) (end 63.500057 132.969002) (layer Edge.Cuts) (width 0.1))
+  (gr_line (start 128.905012 92.964029) (end 128.905012 91.059031) (layer Edge.Cuts) (width 0.1))
+  (gr_line (start 39.370073 61.214051) (end 39.370073 44.704062) (layer Edge.Cuts) (width 0.1))
+  (gr_line (start 147.32 135.509) (end 147.32 122.809009) (layer Edge.Cuts) (width 0.1))
+  (gr_line (start 147.32 96.774027) (end 147.32 109.474018) (layer Edge.Cuts) (width 0.1))
+  (gr_line (start 66.040055 96.774027) (end 66.040055 97.409026) (layer Edge.Cuts) (width 0.1))
+  (gr_line (start 40.640072 61.214051) (end 39.370073 61.214051) (layer Edge.Cuts) (width 0.1))
+  (gr_line (start 141.622783 17.399081) (end 73.66005 17.399081) (layer Edge.Cuts) (width 0.1))
+  (gr_line (start 83.185043 96.774027) (end 83.185043 109.474018) (layer Edge.Cuts) (width 0.1))
+  (gr_line (start 128.905012 96.774027) (end 143.510002 96.774027) (layer Edge.Cuts) (width 0.1))
+  (gr_line (start 80.645045 96.774027) (end 68.580053 96.774027) (layer Edge.Cuts) (width 0.1))
+  (gr_line (start 176.52998 96.774027) (end 147.32 96.774027) (layer Edge.Cuts) (width 0.1))
+  (gr_line (start 176.52998 92.964029) (end 176.52998 91.059031) (layer Edge.Cuts) (width 0.1))
+  (gr_line (start 147.32 122.809009) (end 146.05 122.809009) (layer Edge.Cuts) (width 0.1))
+  (gr_line (start 147.32 39.624066) (end 141.622783 39.624066) (layer Edge.Cuts) (width 0.1))
+  (gr_line (start 45.720069 161.543983) (end 45.720069 148.843991) (layer Edge.Cuts) (width 0.1))
+  (gr_line (start 63.500057 91.059031) (end 31.750078 91.059031) (layer Edge.Cuts) (width 0.1))
+  (gr_line (start 143.510002 148.843991) (end 147.32 148.843991) (layer Edge.Cuts) (width 0.1))
+  (gr_line (start 68.580053 96.774027) (end 66.040055 96.774027) (layer Edge.Cuts) (width 0.1))
+  (gr_line (start 74.295049 39.624066) (end 71.120051 39.624066) (layer Edge.Cuts) (width 0.1))
+  (gr_line (start 83.185043 96.774027) (end 93.980036 96.774027) (layer Edge.Cuts) (width 0.1))
+  (gr_line (start 83.185043 109.474018) (end 80.645045 109.474018) (layer Edge.Cuts) (width 0.1))
+  (gr_line (start 39.370073 44.704062) (end 64.770056 44.704062) (layer Edge.Cuts) (width 0.1))
+  (gr_line (start 147.32 109.474018) (end 143.510002 109.474018) (layer Edge.Cuts) (width 0.1))
+  (gr_line (start 63.500057 161.543983) (end 45.720069 161.543983) (layer Edge.Cuts) (width 0.1))
+  (gr_line (start 176.52998 91.059031) (end 147.32 91.059031) (layer Edge.Cuts) (width 0.1))
+  (gr_line (start 141.605004 91.059031) (end 141.605004 67.564047) (layer Edge.Cuts) (width 0.1))
+  (gr_line (start 66.040055 96.774027) (end 66.040055 109.474018) (layer Edge.Cuts) (width 0.1))
+  (gr_line (start 63.500057 109.474018) (end 63.500057 96.774027) (layer Edge.Cuts) (width 0.1))
+  (gr_line (start 116.205021 96.774027) (end 116.205021 92.964029) (layer Edge.Cuts) (width 0.1))
+  (gr_line (start 66.040055 148.843991) (end 63.500057 148.843991) (layer Edge.Cuts) (width 0.1))
+  (gr_line (start 45.720069 132.969002) (end 45.720069 134.239001) (layer Edge.Cuts) (width 0.1))
+  (gr_line (start 74.295049 67.564047) (end 71.120051 67.564047) (layer Edge.Cuts) (width 0.1))
+  (gr_line (start 189.229971 92.964029) (end 189.229971 91.059031) (layer Edge.Cuts) (width 0.1))
+  (gr_line (start 64.770056 61.214051) (end 40.640072 61.214051) (layer Edge.Cuts) (width 0.1))
+  (gr_line (start 147.32 148.843991) (end 147.32 161.543983) (layer Edge.Cuts) (width 0.1))
+  (gr_line (start 30.480079 86.614034) (end 30.480079 29.464073) (layer Edge.Cuts) (width 0.1))
+  (gr_line (start 147.32 161.543983) (end 214.629954 161.543983) (layer Edge.Cuts) (width 0.1))
+  (gr_line (start 213.359955 96.774027) (end 214.629954 96.774027) (layer Edge.Cuts) (width 0.1))
+  (gr_line (start 83.185043 148.843991) (end 80.645045 148.843991) (layer Edge.Cuts) (width 0.1))
+  (gr_line (start 189.229971 92.964029) (end 189.229971 96.774027) (layer Edge.Cuts) (width 0.1))
+  (gr_line (start 189.229971 96.774027) (end 213.359955 96.774027) (layer Edge.Cuts) (width 0.1))
+  (gr_line (start 143.510002 135.509) (end 143.510002 122.809009) (layer Edge.Cuts) (width 0.1))
+  (gr_line (start 63.500057 132.969002) (end 66.040055 132.969002) (layer Edge.Cuts) (width 0.1))
+  (gr_line (start 63.500057 118.999012) (end 45.720069 118.999012) (layer Edge.Cuts) (width 0.1))
+  (gr_line (start 66.040055 132.969002) (end 66.040055 118.999012) (layer Edge.Cuts) (width 0.1))
+  (gr_line (start 57.785061 29.464073) (end 30.480079 29.464073) (layer Edge.Cuts) (width 0.1))
+  (gr_line (start 147.32 39.624066) (end 147.32 17.399081) (layer Edge.Cuts) (width 0.1))
+  (gr_line (start 66.040055 161.543983) (end 66.040055 148.843991) (layer Edge.Cuts) (width 0.1))
+  (gr_line (start 128.905012 91.059031) (end 141.622783 91.059031) (layer Edge.Cuts) (width 0.1))
+  (gr_line (start 146.05 135.509) (end 143.510002 135.509) (layer Edge.Cuts) (width 0.1))
 )

Commit message: Working on the PCB Layout.
Parts:
- added AE1: Antenna_Shield, Antenna:Antenna, F.Cu at (94.4, 102.5)
- added C1, C2: .1 uf, Capacitors_SMD:C_0603, F.Cu at (122.6, 171.6)
- added C10: 4.7uf, Capacitors_SMD:CP_Elec_4x5.7, F.Cu at (71.6, 134.6)
- added C11: 470pf, Capacitors_SMD:C_0402, F.Cu at (84.1, 127.8)
- added C12: 1uf, MyCaps:C_0603_POL, F.Cu at (87.9, 127.3)
- added C13: 22 uf 100V, Capacitors_SMD:CP_Elec_8x10, F.Cu at (191.0, 143.5)
- added C14: 10pf, Capacitors_SMD:C_0402, F.Cu at (91.2, 154.4)
- added C15: 47pf, Capacitors_SMD:C_0402, F.Cu at (93.5, 153.9)
- added C16: 100nf, Capacitors_SMD:C_0402, F.Cu at (86.3, 154.2)
- added C17: 10uf, Capacitors_SMD:C_0805, F.Cu at (94.0, 104.9)
- added C18: 47pf, Capacitors_SMD:C_0402, F.Cu at (94.5, 153.9)
- added C19: 4.7uf, Capacitors_SMD:CP_Elec_4x5.7, F.Cu at (87.1, 150.9)
- added C20: 10uf, Capacitors_SMD:C_0805, F.Cu at (92.1, 104.9)
- added C21: 1uf, Capacitors_SMD:C_0402, F.Cu at (90.6, 105.6)
- added C22: 100nf, Capacitors_SMD:C_0402, F.Cu at (98.0, 107.1)
- added C23: 100nf, Capacitors_SMD:C_0402, F.Cu at (89.5, 105.6)
- added C24: 5.8pf, Capacitors_SMD:C_0402, F.Cu at (97.3, 104.9)
- added C25: 1uf, Capacitors_SMD:C_0402, F.Cu at (100.1, 112.0)
- added C26: 100nf, Capacitors_SMD:C_0402, F.Cu at (105.2, 159.3)
- added C27: 100pf, Capacitors_SMD:C_0402, F.Cu at (100.1, 113.0)
- added C28: 100nf, Capacitors_SMD:C_0402, F.Cu at (89.9, 112.0)
- added C29: 1uf, Capacitors_SMD:C_0402, F.Cu at (107.3, 119.3)
- added C3: .1 uf, Capacitors_SMD:C_0603, F.Cu at (149.9, 117.6)
- added C30: 100nf, Capacitors_SMD:C_0402, F.Cu at (97.3, 117.4)
- added C31: 270pf, Capacitors_SMD:C_0402, F.Cu at (94.1, 107.6)
- added C32: 10nf, Capacitors_SMD:C_0402, F.Cu at (100.6, 109.7)
- added C33: 270pf, Capacitors_SMD:C_0402, F.Cu at (96.2, 107.6)
- added C34: 3nf, Capacitors_SMD:C_0402, F.Cu at (99.1, 109.2)
- added C35: 22pf, Capacitors_SMD:C_0402, F.Cu at (104.9, 108.7)
- added C36: 22pf, Capacitors_SMD:C_0402, F.Cu at (103.4, 113.0)
- added C37: 1uf, Capacitors_SMD:C_0402, F.Cu at (92.2, 117.7)
- added C4: 15 uf 63V, Capacitors_SMD:CP_Elec_4x5.7, F.Cu at (154.4, 111.8)
- added C5: 47 nf, Capacitors_SMD:C_0603, F.Cu at (163.8, 133.9)
- added C6: 10uf, Capacitors_SMD:CP_Elec_4x5.7, F.Cu at (78.0, 113.3)
- added C7: .1uf, Capacitors_SMD:C_0402, F.Cu at (90.5, 137.9)
- added C8: 220 uf 25V, Capacitors_SMD:CP_Elec_8x10, F.Cu at (179.1, 127.8)
- added C9: 4.7uf, Capacitors_SMD:CP_Elec_4x5.7, F.Cu at (68.8, 126.7)
- added D1: Status, APHB1608CGKSURKC:APHB1608CGKSURKC, F.Cu at (32.0, 70.5)
- added D10: LED, LEDs:LED_D5.0mm, F.Cu at (209.6, 81.3)
- added D11: LED, LEDs:LED_D5.0mm, F.Cu at (209.6, 73.7)
- added D12: LED, LEDs:LED_D5.0mm, F.Cu at (209.6, 66.0)
- added D13: LED, LEDs:LED_D5.0mm, F.Cu at (209.6, 58.4)
- added D14: LED, LEDs:LED_D5.0mm, F.Cu at (209.6, 50.8)
- added D15: LED, LEDs:LED_D5.0mm, F.Cu at (209.6, 43.2)
- added D16: LED, LEDs:LED_D5.0mm, F.Cu at (209.6, 35.6)
- added D17: LED, LEDs:LED_D5.0mm, F.Cu at (209.6, 27.9)
- added D18: DFLS240-7, Diodes_SMD:D_PowerDI-123, F.Cu at (200.7, 106.4)
- added D19: DFLS240-7, Diodes_SMD:D_PowerDI-123, F.Cu at (200.7, 154.5)
- added D2: LED, LEDs:LED_D5.0mm, F.Cu at (135.9, 27.9)
- added D20: SMAJ5.0A/TR13, Diodes_SMD:D_SMA, F.Cu at (71.8, 111.8)
- added D21: LED, LEDs:LED_0402, F.Cu at (78.2, 128.5)
- added D22: LED, LEDs:LED_0402, F.Cu at (78.2, 127.3)
- added D23: LED, LEDs:LED_0402, F.Cu at (78.2, 126.0)
- added D24: DFLS240-7, Diodes_SMD:D_PowerDI-123, F.Cu at (92.5, 149.4)
- added D25: DFLS240-7, Diodes_SMD:D_PowerDI-123, F.Cu at (159.8, 141.0)
- added D26: DFLS240-7, Diodes_SMD:D_PowerDI-123, F.Cu at (72.6, 126.5)
- added D27: SB160-E3/54, Diodes_SMD:D_SMB, F.Cu at (196.8, 115.6)
- added D28: ACT2, LEDs:LED_0402, F.Cu at (87.7, 113.8)
- added D29: ACT1, LEDs:LED_0402, F.Cu at (87.7, 112.6)
- added D3: LED, LEDs:LED_D5.0mm, F.Cu at (135.9, 35.6)
- added D4: LED, LEDs:LED_D5.0mm, F.Cu at (135.9, 43.2)
- added D5: LED, LEDs:LED_D5.0mm, F.Cu at (135.9, 50.8)
- added D6: LED, LEDs:LED_D5.0mm, F.Cu at (135.9, 58.4)
- added D7: LED, LEDs:LED_D5.0mm, F.Cu at (135.9, 66.0)
- added D8: LED, LEDs:LED_D5.0mm, F.Cu at (135.9, 73.7)
- added D9: LED, LEDs:LED_D5.0mm, F.Cu at (135.9, 81.3)
- added EN1: Throttle, Encoders:Series25L-Encoder, F.Cu at (48.3, 105.4)
- added EN2: Reverser, Encoders:ALPSEC12C, F.Cu at (53.9, 141.0)
- added FD1, FD2, FD3: FidMark, Fiducials:Fiducial_1mm_Dia_2.54mm_Outer_CopperBottom, F.Cu at (122.6, 171.6)
- added J1: Button & LED Panel, Pin_Headers:Pin_Header_Straight_1x05_Pitch2.54mm, F.Cu at (128.3, 120.7)
- added J10: RJ45, RJ45-8N-S:RJ45_8N-S, F.Cu at (170.8, 152.4)
- added J11: Barrel_Jack, Connectors:BARREL_JACK, F.Cu at (74.0, 107.0)
- added J12: Battery, Connectors_JST:JST_PH_B2B-PH-SM4-TB_02x2.00mm_Straight, F.Cu at (70.1, 142.2)
- added J13: USB_OTG, Connectors_USB:USB_Micro-B_Molex_47346-0001, F.Cu at (94.2, 160.0)
- added J2: Button & LED Panel, Pin_Headers:Pin_Header_Straight_1x05_Pitch2.54mm, F.Cu at (132.1, 120.7)
- added J3: STEMMA (Display), Connectors_JST:JST_PH_B4B-PH-SM4-TB_04x2.00mm_Straight, F.Cu at (138.6, 110.2)
- added J4: Horn, Pin_Headers:Pin_Header_Straight_1x03_Pitch2.54mm, F.Cu at (124.5, 120.7)
- added J5: Brake, Pin_Headers:Pin_Header_Straight_1x03_Pitch2.54mm, F.Cu at (120.7, 120.7)
- added J6: Light Switch, Pin_Headers:Pin_Header_Straight_1x05_Pitch2.54mm, F.Cu at (113.0, 99.1)
- added J7: Reverser, Pin_Headers:Pin_Header_Straight_1x03_Pitch2.54mm, F.Cu at (127.0, 102.9)
- added J8: Throttle, Pin_Headers:Pin_Header_Straight_1x03_Pitch2.54mm, F.Cu at (127.0, 99.1)
- added J9: RJ45, RJ45-8N-S:RJ45_8N-S, F.Cu at (172.1, 105.4)
- added JP1: Termination, Pin_Headers:Pin_Header_Straight_2x02_Pitch2.54mm, F.Cu at (161.3, 127.0)
- added L1: 330 uh, SRN1060:SRN1060, F.Cu at (188.0, 116.8)
- added L2: Ferrite Bead, Inductors_SMD:L_0402, F.Cu at (92.5, 154.5)
- added L4: 2.0nH, Inductors_SMD:L_0402, F.Cu at (96.1, 105.7)
- added MK1: Mounting_Hole, Mounting_Holes:MountingHole_2.5mm, F.Cu at (34.3, 29.8)
- added MK10: Mounting_Hole, Mounting_Holes:MountingHole_2.5mm, F.Cu at (138.4, 20.3)
- added MK11: Mounting_Hole, Mounting_Holes:MountingHole_2.5mm, F.Cu at (138.4, 87.6)
- added MK12: Mounting_Hole, Mounting_Holes:MountingHole_2.5mm, F.Cu at (77.5, 87.6)
- added MK13: Mounting_Hole, Mounting_Holes:MountingHole_2.5mm, F.Cu at (210.8, 20.3)
- added MK14: Mounting_Hole, Mounting_Holes:MountingHole_2.5mm, F.Cu at (210.8, 87.6)
- added MK15: Mounting_Hole, Mounting_Holes:MountingHole_2.5mm, F.Cu at (151.1, 87.6)
- added MK16: Mounting_Hole, Mounting_Holes:MountingHole_2.5mm, F.Cu at (151.1, 20.3)
- added MK17: Mounting_Hole, Mounting_Holes:MountingHole_2.5mm, F.Cu at (86.4, 158.8)
- added MK18: Mounting_Hole, Mounting_Holes:MountingHole_2.5mm, F.Cu at (139.7, 157.5)
- added MK19: Mounting_Hole, Mounting_Holes:MountingHole_2.5mm, F.Cu at (139.7, 100.3)
- added MK2: Mounting_Hole, Mounting_Holes:MountingHole_2.5mm, F.Cu at (67.3, 29.8)
- added MK20: Mounting_Hole_PAD, Mounting_Holes:MountingHole_2.5mm_Pad, F.Cu at (86.4, 100.3)
- added MK21: Mounting_Hole, Mounting_Holes:MountingHole_2.5mm, F.Cu at (35.1, 65.5)
- added MK22: Mounting_Hole, Mounting_Holes:MountingHole_2.5mm, F.Cu at (65.5, 63.5)
- added MK23: Mounting_Hole, Mounting_Holes:MountingHole_2.5mm, F.Cu at (35.1, 35.1)
- added MK24: Mounting_Hole, Mounting_Holes:MountingHole_2.5mm, F.Cu at (65.5, 35.6)
- added MK3: Mounting_Hole, Mounting_Holes:MountingHole_2.5mm, F.Cu at (67.3, 82.5)
- added MK4: Mounting_Hole, Mounting_Holes:MountingHole_2.5mm, F.Cu at (34.3, 82.5)
- added MK5: Mounting_Hole, Mounting_Holes:MountingHole_2.5mm, F.Cu at (35.6, 120.7)
- added MK6: Mounting_Hole, Mounting_Holes:MountingHole_2.5mm, F.Cu at (62.2, 120.7)
- added MK7: Mounting_Hole, Mounting_Holes:MountingHole_2.5mm, F.Cu at (48.3, 152.4)
- added MK8: Mounting_Hole, Mounting_Holes:MountingHole_2.5mm, F.Cu at (61.0, 152.4)
- added MK9: Mounting_Hole, Mounting_Holes:MountingHole_2.5mm, F.Cu at (77.5, 20.3)
- added P1: CONN_8, Pin_Headers:Pin_Header_Angled_1x08_Pitch2.54mm, F.Cu at (58.4, 82.5)
- added P2: Misc buttons, bell, status LED, Pin_Headers:Pin_Header_Straight_1x08_Pitch2.54mm, F.Cu at (114.3, 106.7)
- added P6: CONN_3, Pin_Headers:Pin_Header_Angled_1x03_Pitch2.54mm, F.Cu at (50.8, 119.4)
- added P7: CONN_3, Pin_Headers:Pin_Header_Angled_1x03_Pitch2.54mm, F.Cu at (57.1, 157.5)
- added P8: CONN_5, Pin_Headers:Pin_Header_Angled_1x05_Pitch2.54mm, F.Cu at (78.7, 80.0)
- added P9: CONN_5, Pin_Headers:Pin_Header_Angled_1x05_Pitch2.54mm, F.Cu at (152.4, 80.0)
- added Q1: UMH3N, TO_SOT_Packages_SMD:SOT-363_SC-70-6, F.Cu at (105.0, 145.9)
- added R1: 220 Ohms, Resistors_SMD:R_0603, F.Cu at (105.3, 105.9)
- added R10: 60 Ohms, Resistors_SMD:R_1206, F.Cu at (161.3, 121.7)
- added R11: 60 Ohms, Resistors_SMD:R_1206, F.Cu at (165.1, 121.7)
- added R12: 330K, Resistors_SMD:R_0402, F.Cu at (70.7, 119.6)
- added R13: 110K, Resistors_SMD:R_0402, F.Cu at (70.6, 118.4)
- added R14: 10K, Resistors_SMD:R_0402, F.Cu at (74.6, 116.1)
- added R15: 470, Resistors_SMD:R_0402, F.Cu at (76.2, 128.5)
- added R16: 470, Resistors_SMD:R_0402, F.Cu at (76.2, 127.3)
- added R17: 470, Resistors_SMD:R_0402, F.Cu at (76.2, 126.0)
- added R18: 5K, Resistors_SMD:R_0402, F.Cu at (78.0, 120.9)
- added R19: 2K, Resistors_SMD:R_0402, F.Cu at (78.0, 119.9)
- added R2: 220 Ohms, Resistors_SMD:R_0603, F.Cu at (87.7, 108.8)
- added R20: 10K, Resistors_SMD:R_0402, F.Cu at (72.1, 123.2)
- added R21: 27, Resistors_SMD:R_0402, F.Cu at (95.5, 154.2)
- added R22: 27, Resistors_SMD:R_0402, F.Cu at (96.5, 154.2)
- added R23: 270, Resistors_SMD:R_0402, F.Cu at (85.7, 113.7)
- added R24: 10K, Resistors_SMD:R_0402, F.Cu at (107.2, 120.8)
- added R25: 270, Resistors_SMD:R_0402, F.Cu at (85.7, 112.6)
- added R26: 20K, Resistors_SMD:R_0402, F.Cu at (99.4, 107.4)
- added R27: 2.4K, Resistors_SMD:R_0402, F.Cu at (106.4, 111.1)
- added R28: 49.9, Resistors_SMD:R_0402, F.Cu at (106.9, 112.5)
- added R29: 49.9, Resistors_SMD:R_0402, F.Cu at (107.0, 113.8)
- added R3, R4, R5, R6: 100K Ohms, Resistors_SMD:R_0402, F.Cu at (122.6, 171.6)
- added R30: 2.4K, Resistors_SMD:R_0402, F.Cu at (106.7, 115.3)
- added R7, R8, R9: 10K, Resistors_SMD:R_0402, F.Cu at (122.6, 171.6)
- added RP1, RP2: 330, 48xxP:4816P, F.Cu at (122.6, 171.6)
- added SW1: A, Buttons_Switches_SMD:SW_SPST_EVQQ2, F.Cu at (36.8, 73.7)
- added SW10: SW_PUSH_SMALL, Buttons_Switches_THT:SW_PUSH_6mm, F.Cu at (131.0, 61.0)
- added SW11: SW_PUSH_SMALL, Buttons_Switches_THT:SW_PUSH_6mm, F.Cu at (130.8, 53.3)
- added SW12: SW_PUSH_SMALL, Buttons_Switches_THT:SW_PUSH_6mm, F.Cu at (124.3, 41.2)
- added SW13: SW_PUSH_SMALL, Buttons_Switches_THT:SW_PUSH_6mm, F.Cu at (131.0, 38.1)
- added SW14: SW_PUSH_SMALL, Buttons_Switches_THT:SW_PUSH_6mm, F.Cu at (130.8, 30.5)
- added SW15: SW_PUSH_SMALL, Buttons_Switches_THT:SW_PUSH_6mm, F.Cu at (204.5, 83.8)
- added SW16: SW_PUSH_SMALL, Buttons_Switches_THT:SW_PUSH_6mm, F.Cu at (204.5, 76.2)
- added SW17: SW_PUSH_SMALL, Buttons_Switches_THT:SW_PUSH_6mm, F.Cu at (204.5, 68.6)
- added SW18: SW_PUSH_SMALL, Buttons_Switches_THT:SW_PUSH_6mm, F.Cu at (204.5, 61.0)
- added SW19: SW_PUSH_SMALL, Buttons_Switches_THT:SW_PUSH_6mm, F.Cu at (204.5, 53.3)
- added SW2: B, Buttons_Switches_SMD:SW_SPST_EVQQ2, F.Cu at (45.7, 73.7)
- added SW20: SW_PUSH_SMALL, Buttons_Switches_THT:SW_PUSH_6mm, F.Cu at (204.5, 45.7)
- added SW21: SW_PUSH_SMALL, Buttons_Switches_THT:SW_PUSH_6mm, F.Cu at (204.5, 38.1)
- added SW22: SW_PUSH_SMALL, Buttons_Switches_THT:SW_PUSH_6mm, F.Cu at (204.5, 30.5)
- added SW23: On/Off, Buttons_Switches_SMD:SW_SPDT_CK-JS102011SAQN, F.Cu at (73.4, 159.2)
- added SW24: RESET, PTS647SN70SMTR2LFS:PTS647SM38SMTR2LFS, F.Cu at (109.6, 125.3)
- added SW3: C, Buttons_Switches_SMD:SW_SPST_EVQQ2, F.Cu at (54.6, 73.7)
- added SW4: D, Buttons_Switches_SMD:SW_SPST_EVQQ2, F.Cu at (63.5, 73.7)
- added SW5: Bell, Buttons_Switches_SMD:SW_SPST_EVQQ2, F.Cu at (49.5, 29.8)
- added SW7: SW_PUSH_SMALL, Buttons_Switches_THT:SW_PUSH_6mm, F.Cu at (130.8, 83.8)
- added SW8: SW_PUSH_SMALL, Buttons_Switches_THT:SW_PUSH_6mm, F.Cu at (130.8, 76.2)
- added SW9: SW_PUSH_SMALL, Buttons_Switches_THT:SW_PUSH_6mm, F.Cu at (130.8, 68.6)
- added T1: Buttons, Terminal_Blocks:TerminalBlock_Pheonix_MPT-2.54mm_9pol, F.Cu at (114.3, 22.9)
- added T2: LEDS, Connectors_Terminal_Blocks:TerminalBlock_Pheonix_MPT-2.54mm_9pol, F.Cu at (92.7, 85.1)
- added T3: Buttons, Connectors_Terminal_Blocks:TerminalBlock_Pheonix_MPT-2.54mm_9pol, F.Cu at (190.5, 22.9)
- added T4: LEDS, Connectors_Terminal_Blocks:TerminalBlock_Pheonix_MPT-2.54mm_9pol, F.Cu at (170.2, 85.1)
- added T5: + 15 in -, Terminal_Blocks:TerminalBlock_Pheonix_MPT-2.54mm_2pol, F.Cu at (207.0, 105.4)
- added T6: + 15 out -, Terminal_Blocks:TerminalBlock_Pheonix_MPT-2.54mm_2pol, F.Cu at (207.0, 156.2)
- added U1, U3: MCP23017, Housings_SOIC:SOIC-28W_7.5x17.9mm_Pitch1.27mm, F.Cu at (122.6, 171.6)
- added U10: ESP32-D0WD-V3, ESP32-D0WD-V3:QFN35P500X500X90-49N-D, F.Cu at (94.9, 112.2)
- added U11: W25Q32JVSSIQ, Housings_SOIC:SOIC-8_3.9x4.9mm_Pitch1.27mm, F.Cu at (94.2, 123.4)
- added U2, U4: TBD62083A, Housings_SOIC:SOIC-18W_7.5x11.6mm_Pitch1.27mm, F.Cu at (122.6, 171.6)
- added U5: TCAN332DR, Housings_SOIC:SOIC-8_3.9x4.9mm_Pitch1.27mm, F.Cu at (154.8, 117.5)
- added U6: MCP73871, Housings_DFN_QFN:QFN-20-1EP_4x4mm_Pitch0.5mm, F.Cu at (74.4, 120.1)
- added U7: LM2574HVM-5.0, SOIC_Wide:SOIC-14_7.4x8.7mm_Pitch1.27mm, F.Cu at (191.1, 128.3)
- added U8: TC1263-3.3VOATR, Housings_SOIC:SO-8_5.3x6.2mm_Pitch1.27mm, F.Cu at (86.0, 134.3)
- added U9: FT231XS-R, Housings_SSOP:SSOP-20_5.3x7.2mm_Pitch0.65mm, F.Cu at (105.1, 153.8)
- added Y1: 40 Mhz +/- 10 ppm, FA_20H:FA20_H, F.Cu at (103.5, 110.8)
Routing:
- net +5V: track 0.00 -> 191.2 mm, vias 0 -> 5
- net GND: track 0.00 -> 184.9 mm, vias 0 -> 47
- net +12V: track 0.00 -> 123.3 mm, vias 0 -> 4
- net /L_Ditch: track 0.00 -> 107.5 mm, vias 0 -> 7
- net /CAN_RX: track 0.00 -> 99.5 mm, vias 0 -> 4
- net /CAN_TX: track 0.00 -> 99.3 mm, vias 0 -> 4
- net /Reverser: track 0.00 -> 82.2 mm, vias 0 -> 4
- net Net-(P2-Pad8): track 0.00 -> 81.5 mm, vias 0 -> 5
- net /L_Bright: track 0.00 -> 68.9 mm, vias 0 -> 4
- net /CAN Transceiver/CANH: track 0.00 -> 61.9 mm, vias 0 -> 4
- net /RST: track 0.00 -> 61.6 mm, vias 0 -> 2
- net /Processor Section/TX: track 0.00 -> 58.1 mm, vias 0 -> 4
- net Net-(C8-Pad1): track 0.00 -> 52.5 mm, vias 0 -> 2
- net /CAN Transceiver/CANL: track 0.00 -> 52.2 mm, vias 0 -> 4
- net Net-(C10-Pad1): track 0.00 -> 47.0 mm, vias 0 -> 4
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- added copper zone on F.Cu, net +3.3V
- added copper zone on B.Cu, net GND
Other:
- outline, holes or cut-outs redrawn
- net class Default: clearance 0.2 -> 0.15
- rule trace_clearance: 0.2 -> 0.15
- rule trace_min: 0.2 -> 0.12
- board text added: "Adafruit 1.3" 128x64 STEMMA OLED"

Commit message: Completed V0.0 PCB.
Parts:
- moved U3 142.1 mm to (173.6, 39.0), turned to 270 degrees
- moved C2 138.7 mm to (162.4, 38.7), turned to 90 degrees
- moved C1 134.7 mm to (86.7, 41.8), turned to 90 degrees
- moved R9 133.9 mm to (169.2, 46.0), turned to 90 degrees
- moved R8 132.6 mm to (165.4, 46.1), turned to 90 degrees
- moved U1 131.9 mm to (97.7, 42.0), turned to 270 degrees
- moved U4 131.3 mm to (176.8, 52.1), turned to 270 degrees
- moved R7 126.0 mm to (93.3, 49.1), turned to 90 degrees
- moved RP2 120.8 mm to (177.4, 63.9), turned to 180 degrees
- moved FD3 120.0 mm to (87.4, 56.9)
- moved U2 118.9 mm to (100.9, 54.7), turned to 270 degrees
- moved RP1 107.5 mm to (101.5, 66.2), turned to 180 degrees
- moved FD2 100.4 mm to (205.7, 115.3)
- moved R4 70.2 mm to (117.3, 101.6)
- moved R6 70.1 mm to (119.2, 101.6)
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Connections:
- C1 pad 2: +3.3V -> +3V3
- C12 pad 1: +3.3V -> +3V3
- C2 pad 2: +3.3V -> +3V3
- C3 pad 1: +3.3V -> +3V3
- C4 pad 1: +3.3V -> +3V3
- J1 pad 2: +3.3V -> +3V3
- J2 pad 2: +3.3V -> +3V3
- J4 pad 1: +3.3V -> +3V3
- J5 pad 1: +3.3V -> +3V3
- P8 pad 2: +3.3V -> +3V3
- P9 pad 2: +3.3V -> +3V3
- R4 pad 1: +3.3V -> +3V3
- R5 pad 1: +3.3V -> +3V3
- R7 pad 1: +3.3V -> +3V3
- R8 pad 1: +3.3V -> +3V3
- R9 pad 1: +3.3V -> +3V3
- U1 pad 9: +3.3V -> +3V3
- U3 pad 9: +3.3V -> +3V3
- U5 pad 3: +3.3V -> +3V3
- U8 pad 1: +3.3V -> +3V3
Routing:
- net GND: track 184.9 -> 587.8 mm, vias 47 -> 64
- net +BATT: track 0.00 -> 285.1 mm, vias 0 -> 2
- net +3V3: track 35.4 -> 205.9 mm, vias 4 -> 15
- net Net-(D17-Pad2): track 0.00 -> 101.2 mm, vias 0 -> 3
- net Net-(D2-Pad2): track 0.00 -> 100.5 mm, vias 0 -> 3
- net Net-(P1-Pad6): track 0.00 -> 94.9 mm, vias 0 -> 4
- net Net-(D3-Pad2): track 0.00 -> 88.9 mm, vias 0 -> 3
- net Net-(D16-Pad2): track 0.00 -> 88.9 mm, vias 0 -> 3
- net Net-(SW7-Pad1): track 0.00 -> 87.6 mm, vias 0 -> 3
- net Net-(D4-Pad2): track 0.00 -> 86.3 mm, vias 0 -> 3
- net Net-(SW8-Pad1): track 0.00 -> 84.3 mm, vias 0 -> 3
- net Net-(SW15-Pad1): track 0.00 -> 83.4 mm, vias 0 -> 3
- net Net-(SW9-Pad1): track 0.00 -> 81.5 mm, vias 0 -> 3
- net Net-(D15-Pad2): track 0.00 -> 80.2 mm, vias 0 -> 3
- net Net-(SW16-Pad1): track 0.00 -> 79.7 mm, vias 0 -> 3
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- added copper zone on F.Cu, net +3V3
- removed copper zone on F.Cu, net +3.3V

Commit message: Started on V0.1 PCB.
Parts:
- moved MK1 223.1 mm to (134.8, 228.4)
- moved MK13 221.6 mm to (134.8, 228.4)
- moved MK23 217.1 mm to (134.8, 228.4)
- moved SW5 216.1 mm to (134.8, 228.4), turned to 0 degrees
- moved MK9 215.9 mm to (134.8, 228.4)
- moved D17 214.0 mm to (134.8, 228.4)
- moved T3 213.0 mm to (134.8, 228.4), turned to 0 degrees
- moved MK2 210.4 mm to (134.8, 228.4)
- moved SW22 209.9 mm to (134.8, 228.4), turned to 0 degrees
- moved MK16 208.8 mm to (134.8, 228.4)
- moved MK10 208.2 mm to (134.8, 228.4)
- moved D16 206.9 mm to (134.8, 228.4)
- moved T1 206.6 mm to (134.8, 228.4), turned to 0 degrees
- moved MK24 204.9 mm to (134.8, 228.4)
- moved SW21 202.7 mm to (134.8, 228.4), turned to 0 degrees
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Routing:
- net GND: track 587.8 -> 32.4 mm, vias 64 -> 25
- net +BATT: track 285.1 -> 0.00 mm, vias 2 -> 0
- net +5V: track 195.4 -> 0.00 mm, vias 5 -> 0
- net +3V3: track 205.9 -> 34.0 mm, vias 15 -> 2
- net +12V: track 129.9 -> 0.00 mm, vias 4 -> 0
- net /L_Ditch: track 106.7 -> 1.20 mm, vias 7 -> 1
- net Net-(D17-Pad2): track 101.2 -> 0.00 mm, vias 3 -> 0
- net Net-(D2-Pad2): track 100.5 -> 0.00 mm, vias 3 -> 0
- net /CAN_RX: track 97.6 -> 0.48 mm, vias 6 -> 1
- net Net-(P1-Pad6): track 94.9 -> 0.00 mm, vias 4 -> 0
- net /CAN_TX: track 100.8 -> 6.65 mm, vias 4 -> 1
- net Net-(D3-Pad2): track 88.9 -> 0.00 mm, vias 3 -> 0
- net Net-(D16-Pad2): track 88.9 -> 0.00 mm, vias 3 -> 0
- net Net-(SW7-Pad1): track 87.6 -> 0.00 mm, vias 3 -> 0
- net Net-(D4-Pad2): track 86.3 -> 0.00 mm, vias 3 -> 0
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Other:
- board outline removed
- rule pad_to_mask_clearance: 0.2 -> 0
- board text removed: "Adafruit 1.3" 128x64 STEMMA OLED"

Commit message: About halfway done.
Parts:
- moved T6 161.7 mm to (242.6, 108.0), turned to 90 degrees
- moved D19 157.7 mm to (242.6, 113.3), turned to 90 degrees
- moved J9 141.9 mm to (207.6, 106.7), turned to 180 degrees
- moved L1 141.5 mm to (227.5, 121.5)
- moved D27 140.9 mm to (238.6, 133.2), turned to 90 degrees
- moved P7 139.5 mm to (54.6, 114.3), turned to 180 degrees
- moved D18 139.0 mm to (242.6, 140.7), turned to 90 degrees
- moved MK7 135.8 mm to (78.7, 104.8)
- moved EN2 135.4 mm to (67.3, 111.0), turned to 270 degrees
- moved U7 134.7 mm to (230.4, 133.6), turned to 90 degrees
- moved T5 134.1 mm to (242.6, 148.6), turned to 90 degrees
- moved MK19 130.3 mm to (174.0, 104.1)
- moved C5 130.1 mm to (194.1, 112.6), turned to 90 degrees
- moved MK5 129.3 mm to (54.6, 127.0)
- moved C8 127.8 mm to (230.6, 143.9)
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Routing:
- net +5V: track 0.00 -> 253.8 mm, vias 0 -> 16
- net GND: track 32.4 -> 207.5 mm, vias 25 -> 49
- net +12V: track 0.00 -> 99.1 mm, vias 0 -> 5
- net /Button_A: track 4.30 -> 67.7 mm, vias 0 -> 3
- net /CAN Transceiver/CANH: track 0.00 -> 52.4 mm, vias 0 -> 3
- net /Processor Section/RX: track 0.00 -> 47.1 mm, vias 0 -> 6
- net Net-(C6-Pad1): track 0.00 -> 46.7 mm, vias 0 -> 4
- net /CAN_TX: track 6.65 -> 53.2 mm, vias 1 -> 4
- net /CAN Transceiver/CANL: track 0.00 -> 45.9 mm, vias 0 -> 3
- net Net-(C9-Pad1): track 0.00 -> 42.1 mm, vias 0 -> 4
- net /CAN_RX: track 0.48 -> 41.8 mm, vias 1 -> 2
- net /L_Dim: track 2.70 -> 43.8 mm, vias 1 -> 4
- net /SDA: track 5.83 -> 46.7 mm, vias 0 -> 1
- net VBUS: track 0.00 -> 38.4 mm, vias 0 -> 5
- net /SCL: track 4.77 -> 41.8 mm, vias 0 -> 1
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Other:
- board outline added: 198.1 x 54 mm

Commit message: Nearly done.  Just the button/LED boards to do.
Parts:
- added REF**: 128x64OLEDSTEMMA, AdafruitDisplays:128x64OLEDSTEMMA, F.Cu at (76.8, 77.5)
- moved MK1 207.2 mm to (55.9, 36.8)
- moved P1 203.2 mm to (67.3, 36.8), turned to 90 degrees
- moved MK2 195.2 mm to (97.8, 36.8)
- moved SW5 194.3 mm to (76.2, 43.2)
- moved D1 190.4 mm to (88.5, 43.8), turned to 270 degrees
- moved SW4 188.6 mm to (64.8, 53.3), turned to 90 degrees
- moved SW3 185.9 mm to (72.4, 53.3), turned to 90 degrees
- moved SW2 183.5 mm to (80.0, 53.3), turned to 90 degrees
- moved SW1 181.3 mm to (87.6, 53.3), turned to 90 degrees
- moved MK3 155.9 mm to (55.9, 94.0)
- moved MK4 139.5 mm to (97.8, 94.0)
Routing:
- net Net-(P1-Pad2): track 0.00 -> 39.6 mm, vias 0 -> 2
- net GND: track 207.5 -> 242.8 mm, vias 49 -> 58
- net Net-(P1-Pad5): track 0.00 -> 30.6 mm, vias 0 -> 2
- net Net-(P1-Pad3): track 0.00 -> 29.8 mm, vias 0 -> 2
- net Net-(P1-Pad4): track 0.00 -> 20.1 mm
- net Net-(P1-Pad6): track 0.00 -> 19.7 mm, vias 0 -> 2
- net Net-(D1-Pad1): track 0.00 -> 16.1 mm, vias 0 -> 2
- net Net-(D1-Pad3): track 0.00 -> 13.2 mm, vias 0 -> 2
Other:
- board size 198.1 x 54 mm -> 198.1 x 121.9 mm
