File: ESP32-D0WD-V3-ControlStand/ESP32-D0WD-V3-ControlStand.sch (KiCad schematic (older format))
At the start: 43 parts, among them J1 Button & LED Panel, J2 Button & LED Panel, J3 STEMMA (Display), J4 Horn, J5 Brake, J6 Light Switch, J7 Reverser, J8 Throttle, P1 CONN_8, P2 Misc buttons, bell, status LED, P3 CONN_3, P4 CONN_3, P5 CONN_5, P6 CONN_3, P7 CONN_3, SW1 A, SW2 B, SW3 C, SW4 D, SW5 Bell, SW6 LIGHT_SWITCH

Commit message: Completed V0-1 board -- added logos, cleaned up silk, added connector labels, etc.
Parts:
- FD1, FD2, FD3: footprint Fiducials:Fiducial_1mm_Dia_2.54mm_Outer_CopperBottom -> Fiducials:Fiducial_1mm_Dia_2.54mm_Outer_CopperTop
Changed lines of the file:
@@
 F 0 "FD1" H 4650 1350 50  0000 C CNN
 F 1 "FidMark" H 4650 1275 50  0000 C CNN
-F 2 "Fiducials:Fiducial_1mm_Dia_2.54mm_Outer_CopperBottom" H 4650 1150 50  0001 C CNN
+F 2 "Fiducials:Fiducial_1mm_Dia_2.54mm_Outer_CopperTop" H 4650 1150 50  0001 C CNN
 F 3 "" H 4650 1150 50  0001 C CNN
 	1    4650 1150
@@
 F 0 "FD2" H 5150 1300 50  0000 C CNN
 F 1 "FidMark" H 5150 1225 50  0000 C CNN
-F 2 "Fiducials:Fiducial_1mm_Dia_2.54mm_Outer_CopperBottom" H 5150 1100 50  0001 C CNN
+F 2 "Fiducials:Fiducial_1mm_Dia_2.54mm_Outer_CopperTop" H 5150 1100 50  0001 C CNN
 F 3 "" H 5150 1100 50  0001 C CNN
 	1    5150 1100
@@
 F 0 "FD3" H 5800 1350 50  0000 C CNN
 F 1 "FidMark" H 5800 1275 50  0000 C CNN
-F 2 "Fiducials:Fiducial_1mm_Dia_2.54mm_Outer_CopperBottom" H 5800 1150 50  0001 C CNN
+F 2 "Fiducials:Fiducial_1mm_Dia_2.54mm_Outer_CopperTop" H 5800 1150 50  0001 C CNN
 F 3 "" H 5800 1150 50  0001 C CNN
 	1    5800 1150
