File: ESP32-S3-WROOM-ControlStand/ESP32-S3-WROOM-ControlStand.kicad_sch (KiCad schematic)
At the start: 42 parts, among them J101 Keypad Panel, J3 Display, J4 Horn, J5 Brake, J6 Light Switch, J7 Reverser, J8 Throttle, P1 To Main Board, P2 Misc buttons, bell, status LED, P3 To Main Board, P4 To Main Board, P5 To Main Board, P6 To Main Board, P7 To Main Board, SW1 A, SW2 B, SW3 C, SW4 D, SW5 Bell, SW6 LIGHT_SWITCH

Commit message: 3D models mostly done.
Parts:
- J3: footprint Connectors_JST:JST_PH_B4B-PH-SM4-TB_04x2.00mm_Straight -> Connector_JST:JST_PH_B4B-PH-K_1x04_P2.00mm_Vertical
- R1, R2: footprint Resistors_SMD:R_0603 -> Resistor_SMD:R_0603_1608Metric
- R3, R4, R5, R6: footprint Resistors_SMD:R_0402 -> Resistor_SMD:R_0402_1005Metric
- SW1, SW2, SW3, SW4, SW5: footprint Buttons_Switches_SMD:SW_SPST_EVQQ2 -> Button_Switch_SMD:SW_SPST_EVQQ2
