File: ESP32-S3-WROOM-ControlStand/KeypadPanel.kicad_sch (KiCad schematic)
At the start: 20 parts, among them P701 To Main Board, SW701 "1", SW702 "4", SW703 "7", SW704 "*", SW705 "2", SW706 "5", SW707 "8", SW708 "0", SW709 "3", SW710 "6", SW711 "9", SW712 "#", U701 TCA8418

Commit message: 3D models mostly done.
Parts:
- C701: footprint Capacitors_SMD:C_0603 -> Capacitor_SMD:C_0603_1608Metric
- R701: footprint Resistors_SMD:R_0603 -> Resistor_SMD:R_0603_1608Metric
- SW701: footprint Buttons_Switches_SMD:SW_SPST_B3U-1100P-B -> Button_Switch_SMD:SW_SPST_B3U-1100P-B
- U701: footprint Housings_DFN_QFN:QFN-24-1EP_4x4mm_Pitch0.5mm -> Package_DFN_QFN:QFN-24-1EP_4x4mm_P0.5mm_EP2.7x2.7mm_ThermalVias
Changed lines of the file:
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@@
       (effects (font (size 1.27 1.27)) (justify left))
     )
-    (property "Footprint" "Housings_DFN_QFN:QFN-24-1EP_4x4mm_Pitch0.5mm" (id 2) (at 109.22 95.885 0)
+    (property "Footprint" "Package_DFN_QFN:QFN-24-1EP_4x4mm_P0.5mm_EP2.7x2.7mm_ThermalVias" (id 2) (at 109.22 95.885 0)
       (effects (font (size 1.27 1.27)) hide)
     )
@@
       (effects (font (size 1.27 1.27)) (justify left))
     )
-    (property "Footprint" "Capacitors_SMD:C_0603" (id 2) (at 93.345 51.1302 0)
+    (property "Footprint" "Capacitor_SMD:C_0603_1608Metric" (id 2) (at 93.345 51.1302 0)
       (effects (font (size 1.27 1.27)) hide)
     )
@@
     (property "Reference" "R701" (id 0) (at 64.77 69.977 90))
     (property "Value" "10K" (id 1) (at 64.77 67.945 90))
-    (property "Footprint" "Resistors_SMD:R_0603" (id 2) (at 64.77 66.167 90)
+    (property "Footprint" "Resistor_SMD:R_0603_1608Metric" (id 2) (at 64.77 66.167 90)
       (effects (font (size 1.27 1.27)) hide)
     )
@@
       (effects (font (size 0.762 0.762)))
     )
-    (property "Footprint" "Buttons_Switches_SMD:SW_SPST_B3U-1100P-B" (id 2) (at 125.73 57.785 0)
+    (property "Footprint" "Button_Switch_SMD:SW_SPST_B3U-1100P-B" (id 2) (at 125.73 57.785 0)
       (effects (font (size 1.524 1.524)) hide)
     )

Commit message: Finalize part numbers for BOM.
Parts:
- U701: Mouser Part Number (none) -> 595-TCA8418RTWR
Changed lines of the file:
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@@
     )
     (property "Datasheet" "" (id 3) (at 85.09 66.675 0))
+    (property "Mouser Part Number" "595-TCA8418RTWR" (id 4) (at 83.82 73.025 0)
+      (effects (font (size 1.27 1.27)) hide)
+    )
     (pin "1")
     (pin "10")
