File: ESP32-S3-WROOM-ControlStand/PowerSupply.kicad_sch (KiCad schematic)
At the start: 26 parts, among them J11 Barrel_Jack, J12 Battery, SW23 On/Off, U6 MCP73871, U8 TC1263-3.3VOATR

Commit message: 3D models mostly done.
Parts:
- C10, C6, C9: footprint Capacitors_SMD:CP_Elec_4x5.7 -> Capacitor_SMD:CP_Elec_4x5.7
- J12: footprint Connectors_JST:JST_PH_B2B-PH-SM4-TB_02x2.00mm_Straight -> Connector_JST:JST_PH_B2B-PH-K_1x02_P2.00mm_Vertical
- U6: footprint Housings_DFN_QFN:QFN-20-1EP_4x4mm_Pitch0.5mm -> Package_DFN_QFN:QFN-20-1EP_4x4mm_P0.5mm_EP2.5x2.5mm_ThermalVias
- U8: footprint Housings_SOIC:SO-8_5.3x6.2mm_Pitch1.27mm -> Package_SO:SOIC-8W_5.3x5.3mm_P1.27mm
Changed lines of the file:
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@@
       (effects (font (size 1.27 1.27)) (justify left))
     )
-    (property "Footprint" "Housings_SOIC:SO-8_5.3x6.2mm_Pitch1.27mm" (id 2) (at 113.03 116.84 0)
+    (property "Footprint" "Package_SO:SOIC-8W_5.3x5.3mm_P1.27mm" (id 2) (at 113.03 116.84 0)
       (effects (font (size 1.27 1.27)) (justify left) hide)
     )
@@
     (property "Reference" "J12" (id 0) (at 120.65 146.05 0))
     (property "Value" "Battery" (id 1) (at 120.65 153.67 0))
-    (property "Footprint" "Connectors_JST:JST_PH_B2B-PH-SM4-TB_02x2.00mm_Straight" (id 2) (at 120.65 148.59 0)
+    (property "Footprint" "Connector_JST:JST_PH_B2B-PH-K_1x02_P2.00mm_Vertical" (id 2) (at 120.65 148.59 0)
       (effects (font (size 1.27 1.27)) hide)
     )
@@
       (effects (font (size 1.524 1.524)))
     )
-    (property "Footprint" "Housings_DFN_QFN:QFN-20-1EP_4x4mm_Pitch0.5mm" (id 2) (at 85.09 153.67 0)
+    (property "Footprint" "Package_DFN_QFN:QFN-20-1EP_4x4mm_P0.5mm_EP2.5x2.5mm_ThermalVias" (id 2) (at 85.09 153.67 0)
       (effects (font (size 1.524 1.524)) hide)
     )
@@
       (effects (font (size 1.27 1.27)) (justify left))
     )
-    (property "Footprint" "Capacitors_SMD:CP_Elec_4x5.7" (id 2) (at 38.1 134.62 0)
+    (property "Footprint" "Capacitor_SMD:CP_Elec_4x5.7" (id 2) (at 38.1 134.62 0)
       (effects (font (size 1.27 1.27)) hide)
     )
@@
       (effects (font (size 1.27 1.27)) (justify left))
     )
-    (property "Footprint" "Capacitors_SMD:CP_Elec_4x5.7" (id 2) (at 105.41 139.7 0)
+    (property "Footprint" "Capacitor_SMD:CP_Elec_4x5.7" (id 2) (at 105.41 139.7 0)
       (effects (font (size 1.27 1.27)) hide)
     )
@@
       (effects (font (size 1.27 1.27)) (justify left))
     )
-    (property "Footprint" "Capacitors_SMD:CP_Elec_4x5.7" (id 2) (at 111.76 154.94 0)
-      (effects (font (size 1.27 1.27)) hide)
-    )
+    (property "Footprint" "Capacitor_SMD:CP_Elec_4x5.7" (id 2) (at 111.76 154.94 0)
+      (effects (font (size 1.27 1.27)) hide)
+    )

Commit message: Finalize part numbers for BOM.
Parts:
- J12: Manufacturer_Name (none) -> JST; Manufaturer_Name JST -> (none)
Changed lines of the file:
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@@
       (effects (font (size 1.27 1.27)) hide)
     )
-    (property "Manufaturer_Name" "JST" (id 4) (at 120.65 148.59 0)
+    (property "Manufacturer_Name" "JST" (id 4) (at 120.65 148.59 0)
       (effects (font (size 1.524 1.524)) hide)
     )
